File: Hardware/Neural_Interface.kicad_pcb (KiCad board)
At the start: 2 copper layers, 0 parts

Commit message: Start Layout
Parts:
- added C1: 1u, Capacitor_SMD:C_0603_1608Metric, F.Cu at (126.8, 30.5)
- added C10: 1u, Capacitor_SMD:C_0603_1608Metric, F.Cu at (148.9, 39.1)
- added C11: 47n, Capacitor_SMD:C_0402_1005Metric, F.Cu at (151.7, 44.5)
- added C12: 470n, Capacitor_SMD:C_0603_1608Metric, F.Cu at (153.0, 44.5)
- added C13: 10n, Capacitor_SMD:C_0402_1005Metric, F.Cu at (154.3, 44.5)
- added C14: 10u, Capacitor_SMD:C_0805_2012Metric, F.Cu at (156.7, 45.5)
- added C15: 10u, Capacitor_SMD:C_0805_2012Metric, F.Cu at (156.7, 47.6)
- added C16: 1u, Capacitor_SMD:C_0603_1608Metric, F.Cu at (156.5, 43.8)
- added C17: 82n, Capacitor_SMD:C_1206_3216Metric, F.Cu at (159.7, 37.0)
- added C18: 820p, Capacitor_SMD:C_0402_1005Metric, F.Cu at (157.9, 39.8)
- added C19: 10u, Capacitor_SMD:C_0805_2012Metric, F.Cu at (159.3, 69.0)
- added C2: 100n, Capacitor_SMD:C_0402_1005Metric, F.Cu at (107.2, 36.2)
- added C20: 1u, Capacitor_SMD:C_0603_1608Metric, F.Cu at (144.6, 70.1)
- added C21: 1u, Capacitor_SMD:C_0603_1608Metric, F.Cu at (159.5, 65.6)
- added C22: 10u, Capacitor_SMD:C_0805_2012Metric, F.Cu at (146.9, 70.3)
- added C23: 10u, Capacitor_SMD:C_0805_2012Metric, F.Cu at (78.8, 87.8)
- added C24: 10u, Capacitor_SMD:C_0805_2012Metric, F.Cu at (118.8, 81.2)
- added C25: 10u, Capacitor_SMD:C_0805_2012Metric, F.Cu at (78.8, 80.4)
- added C26: 10u, Capacitor_SMD:C_0805_2012Metric, F.Cu at (118.8, 64.1)
- added C27: 10u, Capacitor_SMD:C_0805_2012Metric, F.Cu at (124.5, 69.2)
- added C28: 10n, Capacitor_SMD:C_0402_1005Metric, F.Cu at (73.7, 82.0)
- added C29: 10u, Capacitor_SMD:C_0805_2012Metric, F.Cu at (76.5, 80.4)
- added C3: 10u, Capacitor_SMD:C_0805_2012Metric, F.Cu at (105.2, 33.2)
- added C30: 10n, Capacitor_SMD:C_0402_1005Metric, F.Cu at (74.8, 86.1)
- added C31: 100n, Capacitor_SMD:C_0402_1005Metric, F.Cu at (125.1, 89.4)
- added C32: 10u, Capacitor_SMD:C_0805_2012Metric, F.Cu at (76.5, 87.8)
- added C33: 10u, Capacitor_SMD:C_0805_2012Metric, F.Cu at (115.9, 88.6)
- added C34: 10u, Capacitor_SMD:C_0805_2012Metric, F.Cu at (118.8, 83.5)
- added C35: 30p, Capacitor_SMD:C_0402_1005Metric, F.Cu at (38.9, 35.2)
- added C36: 30p, Capacitor_SMD:C_0402_1005Metric, F.Cu at (38.9, 47.4)
- added C37: 30p, Capacitor_SMD:C_0402_1005Metric, F.Cu at (38.9, 59.4)
- added C38: 30p, Capacitor_SMD:C_0402_1005Metric, F.Cu at (38.9, 71.2)
- added C39: 30p, Capacitor_SMD:C_0402_1005Metric, F.Cu at (38.9, 31.4)
- added C4: 100n, Capacitor_SMD:C_0402_1005Metric, F.Cu at (107.2, 34.0)
- added C40: 30p, Capacitor_SMD:C_0402_1005Metric, F.Cu at (38.9, 43.6)
- added C41: 30p, Capacitor_SMD:C_0402_1005Metric, F.Cu at (38.9, 55.6)
- added C42: 30p, Capacitor_SMD:C_0402_1005Metric, F.Cu at (38.9, 67.4)
- added C43: 1u, Capacitor_SMD:C_0603_1608Metric, F.Cu at (42.1, 35.0)
- added C44: 1u, Capacitor_SMD:C_0603_1608Metric, F.Cu at (42.1, 47.2)
- added C45: 1u, Capacitor_SMD:C_0603_1608Metric, F.Cu at (42.1, 59.1)
- added C46: 1u, Capacitor_SMD:C_0603_1608Metric, F.Cu at (42.1, 70.9)
- added C47: 100n, Capacitor_SMD:C_0402_1005Metric, F.Cu at (41.5, 33.6)
- added C48: 100n, Capacitor_SMD:C_0402_1005Metric, F.Cu at (41.5, 45.8)
- added C49: 100n, Capacitor_SMD:C_0402_1005Metric, F.Cu at (41.6, 57.8)
- added C5: 100n, Capacitor_SMD:C_0402_1005Metric, F.Cu at (153.1, 35.3)
- added C50: 100n, Capacitor_SMD:C_0402_1005Metric, F.Cu at (41.6, 69.6)
- added C51: 1u, Capacitor_SMD:C_0603_1608Metric, F.Cu at (45.4, 27.5)
- added C52: 1u, Capacitor_SMD:C_0603_1608Metric, F.Cu at (45.4, 39.7)
- added C53: 1u, Capacitor_SMD:C_0603_1608Metric, F.Cu at (45.5, 51.6)
- added C54: 1u, Capacitor_SMD:C_0603_1608Metric, F.Cu at (45.5, 63.4)
- added C55: 100n, Capacitor_SMD:C_0402_1005Metric, F.Cu at (46.0, 28.8)
- added C56: 100n, Capacitor_SMD:C_0402_1005Metric, F.Cu at (46.0, 41.0)
- added C57: 100n, Capacitor_SMD:C_0402_1005Metric, F.Cu at (46.0, 53.0)
- added C58: 100n, Capacitor_SMD:C_0402_1005Metric, F.Cu at (46.0, 64.8)
- added C59: 30p, Capacitor_SMD:C_0402_1005Metric, F.Cu at (64.6, 44.9)
- added C6: 10n, Capacitor_SMD:C_0402_1005Metric, F.Cu at (153.1, 36.4)
- added C60: 30p, Capacitor_SMD:C_0402_1005Metric, F.Cu at (61.2, 44.9)
- added C61: 30p, Capacitor_SMD:C_0402_1005Metric, F.Cu at (61.2, 54.3)
- added C62: 30p, Capacitor_SMD:C_0402_1005Metric, F.Cu at (64.6, 54.3)
- added C63: 1u, Capacitor_SMD:C_0603_1608Metric, F.Cu at (64.7, 33.3)
- added C64: 100n, Capacitor_SMD:C_0402_1005Metric, F.Cu at (62.8, 29.4)
- added C65: 10u, Capacitor_SMD:C_0805_2012Metric, F.Cu at (62.0, 27.8)
- added C66: 100n, Capacitor_SMD:C_0402_1005Metric, F.Cu at (62.8, 34.3)
- added C67: 1u, Capacitor_SMD:C_0603_1608Metric, F.Cu at (59.6, 48.7)
- added C68: 100n, Capacitor_SMD:C_0402_1005Metric, F.Cu at (63.0, 46.1)
- added C69: 10u, Capacitor_SMD:C_0805_2012Metric, F.Cu at (48.8, 81.3)
- added C7: 470n, Capacitor_SMD:C_0603_1608Metric, F.Cu at (151.4, 35.3)
- added C70: 100n, Capacitor_SMD:C_0402_1005Metric, F.Cu at (47.1, 82.1)
- added C71: 200p, Capacitor_SMD:C_0402_1005Metric, F.Cu at (45.2, 85.7)
- added C72: 10u, Capacitor_SMD:C_0805_2012Metric, F.Cu at (47.6, 91.9)
- added C73: 100n, Capacitor_SMD:C_0402_1005Metric, F.Cu at (46.9, 90.3)
- added C74: 1u, Capacitor_SMD:C_0603_1608Metric, F.Cu at (60.1, 66.7)
- added C75: 1u, Capacitor_SMD:C_0603_1608Metric, F.Cu at (62.6, 70.8)
- added C76: 100n, Capacitor_SMD:C_0402_1005Metric, F.Cu at (62.1, 69.5)
- added C77: 10u, Capacitor_SMD:C_0805_2012Metric, F.Cu at (41.5, 81.1)
- added C78: 1u, Capacitor_SMD:C_0603_1608Metric, F.Cu at (38.6, 83.9)
- added C79: 10u, Capacitor_SMD:C_0805_2012Metric, F.Cu at (51.7, 82.0)
- added C8: 47n, Capacitor_SMD:C_0402_1005Metric, F.Cu at (150.1, 35.9)
- added C80: 100n, Capacitor_SMD:C_0402_1005Metric, F.Cu at (43.1, 80.3)
- added C81: 100n, Capacitor_SMD:C_0402_1005Metric, F.Cu at (52.5, 83.7)
- added C82: 1u, Capacitor_SMD:C_0603_1608Metric, F.Cu at (65.9, 63.3)
- added C83: 100n, Capacitor_SMD:C_0402_1005Metric, F.Cu at (66.5, 64.6)
- added C84: 10u, Capacitor_SMD:C_0805_2012Metric, F.Cu at (81.4, 33.0)
- added C85: 100n, Capacitor_SMD:C_0402_1005Metric, F.Cu at (82.2, 34.7)
- added C86: 1u, Capacitor_SMD:C_0603_1608Metric, F.Cu at (84.0, 31.4)
- added C87: 100n, Capacitor_SMD:C_0402_1005Metric, F.Cu at (85.4, 32.0)
- added C88: 100n, Capacitor_SMD:C_0402_1005Metric, F.Cu at (86.5, 32.0)
- added C89: 1u, Capacitor_SMD:C_0603_1608Metric, F.Cu at (87.9, 31.4)
- added C9: 10n, Capacitor_SMD:C_0402_1005Metric, F.Cu at (155.1, 36.4)
- added D1: MBR130T1G, Diode_SMD:D_SOD-123, F.Cu at (123.2, 81.4)
- added D2: MBR130T1G, Diode_SMD:D_SOD-123, F.Cu at (118.4, 88.0)
- added D3: CDBU0130L-HF, Diode_SMD:D_0603_1608Metric, F.Cu at (65.2, 46.3)
- added D4: CDBU0130L-HF, Diode_SMD:D_0603_1608Metric, F.Cu at (60.6, 46.3)
- added D5: CDBU0130L-HF, Diode_SMD:D_0603_1608Metric, F.Cu at (60.6, 52.9)
- added D6: CDBU0130L-HF, Diode_SMD:D_0603_1608Metric, F.Cu at (65.2, 52.9)
- added IC1: BQ51013BRHLR, Neural_Footprints:BQ51050BRHLR, F.Cu at (153.7, 39.9)
- added IC10: INA823DGKR, Neural_Footprints:SOP65P490X110-8N, F.Cu at (43.8, 55.4)
- added IC11: INA823DGKR, Neural_Footprints:SOP65P490X110-8N, F.Cu at (43.8, 67.2)
- added IC12: REF35160QDBVR, Neural_Footprints:SOT95P280X145-6N, F.Cu at (61.6, 31.8)
- added IC13: LM324LVIDYYR, Neural_Footprints:SOP50P326X110-14N, F.Cu at (62.9, 49.6)
- added IC14: ADA4898-2YRDZ, Neural_Footprints:SOIC127P600X175-9N, F.Cu at (49.7, 87.0)
- added IC15: AD8067ARTZ-REEL7, Neural_Footprints:SOT95P280X145-5N, F.Cu at (45.1, 81.2)
- added IC16: INA823DGKR, Neural_Footprints:SOP65P490X110-8N, F.Cu at (64.3, 67.0)
- added IC17: MCP3464RT-E_NC, Neural_Footprints:QFN40P300X300X60-21N-D, F.Cu at (85.9, 35.3)
- added IC2: CSD75207W15, Neural_Footprints:BGA9C50P3X3_146X146X62, F.Cu at (152.5, 63.0)
- added IC3: BQ25185DLHR, Neural_Footprints:SON40P220X200X80-11N, F.Cu at (161.7, 69.0)
- added IC4: BQ27427YZFR, Neural_Footprints:BGA9C50P3X3_158X162X62, F.Cu at (144.0, 66.4)
- added IC5: TPS7A3901DSCR, Neural_Footprints:SON50P300X300X80-11N-D, F.Cu at (77.7, 84.1)
- added IC6: TLV62585DRLR, Neural_Footprints:SOTFL50P160X60-6N, F.Cu at (124.0, 66.9)
- added IC7: BD8316GWL-E2, Neural_Footprints:BGA11C40P4X3_180X150X55, F.Cu at (124.0, 86.4)
- added IC8: INA823DGKR, Neural_Footprints:SOP65P490X110-8N, F.Cu at (43.8, 31.2)
- added IC9: INA823DGKR, Neural_Footprints:SOP65P490X110-8N, F.Cu at (43.8, 43.4)
- added J1: Conn_02x07_Odd_Even, Connector_PinHeader_2.54mm:PinHeader_2x07_P2.54mm_Vertical, F.Cu at (135.6, 41.2)
- added J10: Conn_01x03, Connector_PinHeader_2.54mm:PinHeader_1x03_P2.54mm_Vertical, F.Cu at (159.8, 75.5)
- added J11: Conn_01x02, Connector_PinHeader_2.54mm:PinHeader_1x02_P2.54mm_Vertical, F.Cu at (110.1, 84.4)
- added J12: Conn_01x02, Connector_PinHeader_2.54mm:PinHeader_1x02_P2.54mm_Vertical, F.Cu at (110.1, 88.3)
- added J13: Conn_01x02, Connector_PinHeader_2.54mm:PinHeader_1x02_P2.54mm_Vertical, F.Cu at (117.8, 74.6)
- added J14: Conn_01x02, Connector_PinHeader_2.54mm:PinHeader_1x02_P2.54mm_Vertical, F.Cu at (65.6, 86.0)
- added J15: Conn_01x02, Connector_PinHeader_2.54mm:PinHeader_1x02_P2.54mm_Vertical, F.Cu at (65.6, 81.9)
- added J16: Conn_01x10, Connector_PinHeader_2.54mm:PinHeader_1x10_P2.54mm_Vertical, F.Cu at (21.8, 56.2)
- added J17: 505110-1092, Neural_Footprints:5051101092, F.Cu at (22.2, 43.1)
- added J18: Conn_01x03, Connector_PinHeader_2.54mm:PinHeader_1x03_P2.54mm_Vertical, F.Cu at (82.2, 46.9)
- added J19: Conn_01x03, Connector_PinHeader_2.54mm:PinHeader_1x03_P2.54mm_Vertical, F.Cu at (82.2, 44.2)
- added J2: Conn_02x06_Odd_Even, Connector_PinSocket_2.54mm:PinSocket_2x06_P2.54mm_Vertical, F.Cu at (86.3, 57.4)
- added J20: Conn_01x03, Connector_PinHeader_2.54mm:PinHeader_1x03_P2.54mm_Vertical, F.Cu at (82.2, 49.5)
- added J21: Conn_01x03, Connector_PinHeader_2.54mm:PinHeader_1x03_P2.54mm_Vertical, F.Cu at (82.2, 52.2)
- added J22: Conn_01x02, Connector_PinHeader_2.54mm:PinHeader_1x02_P2.54mm_Vertical, F.Cu at (105.5, 47.2)
- added J3: Conn_01x05, Connector_PinHeader_2.54mm:PinHeader_1x05_P2.54mm_Vertical, F.Cu at (109.9, 49.6)
- added J4: Conn_01x04, Connector_PinHeader_2.54mm:PinHeader_1x04_P2.54mm_Vertical, F.Cu at (138.2, 28.7)
- added J5: Conn_01x03, Connector_PinHeader_2.54mm:PinHeader_1x03_P2.54mm_Vertical, F.Cu at (155.9, 75.5)
- added J6: Conn_01x02, Connector_PinHeader_2.54mm:PinHeader_1x02_P2.54mm_Vertical, F.Cu at (139.0, 70.4)
- added J7: S2B-PH-SM4-TB, Neural_Footprints:CONN_S2B-PH-SM4-TB_JST, F.Cu at (160.7, 90.5)
- added J8: Conn_01x03, Jumper:SolderJumper-3_P1.3mm_Open_Pad1.0x1.5mm, F.Cu at (162.8, 84.6)
- added J9: Conn_01x03, Jumper:SolderJumper-3_P1.3mm_Open_Pad1.0x1.5mm, F.Cu at (158.1, 84.6)
- added L1: 1uH, Inductor_SMD:L_Coilcraft_XAL4020-XXX, F.Cu at (119.5, 67.8)
- added L2: 4.7uH, Inductor_SMD:L_0603_1608Metric, F.Cu at (124.0, 83.7)
- added L3: 4.7uH, Inductor_SMD:L_0603_1608Metric, F.Cu at (120.5, 87.1)
- added R1: 10k, Resistor_SMD:R_0402_1005Metric, F.Cu at (126.8, 33.5)
- added R10: 5.1k, Resistor_SMD:R_0402_1005Metric, F.Cu at (146.7, 88.9)
- added R11: 10k, Resistor_SMD:R_0402_1005Metric, F.Cu at (147.6, 38.6)
- added R12: 10k, Resistor_SMD:R_0402_1005Metric, F.Cu at (141.0, 67.3)
- added R13: 10k, Resistor_SMD:R_0402_1005Metric, F.Cu at (162.2, 71.6)
- added R14: 10k, Resistor_SMD:R_0402_1005Metric, F.Cu at (141.0, 66.0)
- added R15: 10k, Resistor_SMD:R_0402_1005Metric, F.Cu at (160.9, 65.1)
- added R16: 10k, Resistor_SMD:R_0402_1005Metric, F.Cu at (164.0, 65.1)
- added R17: 130k, Resistor_SMD:R_0402_1005Metric, F.Cu at (162.9, 65.1)
- added R18: 3k, Resistor_SMD:R_0402_1005Metric, F.Cu at (161.9, 65.1)
- added R19: 453k, Resistor_SMD:R_0402_1005Metric, F.Cu at (123.7, 64.9)
- added R2: 10k, Resistor_SMD:R_0402_1005Metric, F.Cu at (104.5, 72.9)
- added R20: 100k, Resistor_SMD:R_0402_1005Metric, F.Cu at (125.7, 64.9)
- added R21: 100k, Resistor_SMD:R_0402_1005Metric, F.Cu at (126.9, 87.3)
- added R22: 10k, Resistor_SMD:R_0402_1005Metric, F.Cu at (126.9, 89.4)
- added R23: 10k, Resistor_SMD:R_0402_1005Metric, F.Cu at (74.1, 83.5)
- added R24: 28k, Resistor_SMD:R_0402_1005Metric, F.Cu at (74.8, 82.0)
- added R25: 17.8k, Resistor_SMD:R_0402_1005Metric, F.Cu at (73.7, 86.1)
- added R26: 10k, Resistor_SMD:R_0402_1005Metric, F.Cu at (74.1, 84.6)
- added R27: 90.9k, Resistor_SMD:R_0402_1005Metric, F.Cu at (123.0, 89.4)
- added R28: 10k, Resistor_SMD:R_0402_1005Metric, F.Cu at (124.1, 89.4)
- added R29: 600k, Resistor_SMD:R_0402_1005Metric, F.Cu at (38.9, 32.7)
- added R3: 10k, Resistor_SMD:R_0402_1005Metric, F.Cu at (105.0, 67.8)
- added R30: 332k, Resistor_SMD:R_0402_1005Metric, F.Cu at (38.9, 34.0)
- added R31: 600k, Resistor_SMD:R_0402_1005Metric, F.Cu at (38.9, 44.9)
- added R32: 332k, Resistor_SMD:R_0402_1005Metric, F.Cu at (38.9, 46.2)
- added R33: 600k, Resistor_SMD:R_0402_1005Metric, F.Cu at (38.9, 56.8)
- added R34: 332k, Resistor_SMD:R_0402_1005Metric, F.Cu at (38.9, 58.1)
- added R35: 600k, Resistor_SMD:R_0402_1005Metric, F.Cu at (38.9, 68.6)
- added R36: 332k, Resistor_SMD:R_0402_1005Metric, F.Cu at (38.9, 69.9)
- added R37: 600k, Resistor_SMD:R_0402_1005Metric, F.Cu at (38.9, 28.8)
- added R38: 332k, Resistor_SMD:R_0402_1005Metric, F.Cu at (38.9, 30.1)
- added R39: 600k, Resistor_SMD:R_0402_1005Metric, F.Cu at (38.9, 41.0)
- added R4: 10k, Resistor_SMD:R_0402_1005Metric, F.Cu at (103.9, 67.8)
- added R40: 332k, Resistor_SMD:R_0402_1005Metric, F.Cu at (38.9, 42.3)
- added R41: 600k, Resistor_SMD:R_0402_1005Metric, F.Cu at (38.9, 53.0)
- added R42: 332k, Resistor_SMD:R_0402_1005Metric, F.Cu at (38.9, 54.3)
- added R43: 600k, Resistor_SMD:R_0402_1005Metric, F.Cu at (38.9, 64.8)
- added R44: 332k, Resistor_SMD:R_0402_1005Metric, F.Cu at (38.9, 66.1)
- added R45: 24.9k, Resistor_SMD:R_0402_1005Metric, F.Cu at (41.5, 28.8)
- added R46: 24.9k, Resistor_SMD:R_0402_1005Metric, F.Cu at (41.6, 41.0)
- added R47: 24.9k, Resistor_SMD:R_0402_1005Metric, F.Cu at (41.6, 53.0)
- added R48: 24.9k, Resistor_SMD:R_0402_1005Metric, F.Cu at (41.6, 64.8)
- added R49: 10k, Resistor_SMD:R_0402_1005Metric, F.Cu at (64.2, 43.3)
- added R5: 330, Resistor_SMD:R_0402_1005Metric, F.Cu at (148.8, 42.6)
- added R50: 10k, Resistor_SMD:R_0402_1005Metric, F.Cu at (61.6, 43.3)
- added R51: 10k, Resistor_SMD:R_0402_1005Metric, F.Cu at (61.6, 55.9)
- added R52: 10k, Resistor_SMD:R_0402_1005Metric, F.Cu at (64.2, 55.9)
- added R53: 82.5k, Resistor_SMD:R_0603_1608Metric, F.Cu at (41.9, 85.5)
- added R54: 82.5k, Resistor_SMD:R_0603_1608Metric, F.Cu at (41.9, 87.2)
- added R55: 100R, Resistor_SMD:R_0402_1005Metric, F.Cu at (44.1, 85.7)
- added R56: 1R, Resistor_SMD:R_0603_1608Metric, F.Cu at (21.7, 83.0)
- added R57: 100R, Resistor_SMD:R_0402_1005Metric, F.Cu at (55.0, 87.7)
- added R58: 2k, Resistor_SMD:R_0402_1005Metric, F.Cu at (45.5, 78.6)
- added R59: 200, Resistor_SMD:R_0402_1005Metric, F.Cu at (62.1, 64.6)
- added R6: 196, Resistor_SMD:R_0402_1005Metric, F.Cu at (149.3, 44.1)
- added R60: 4R, Resistor_SMD:R_0603_1608Metric, F.Cu at (41.9, 83.9)
- added R61: 10R, Resistor_SMD:R_0402_1005Metric, F.Cu at (82.6, 30.9)
- added R62: 10R, Resistor_SMD:R_0402_1005Metric, F.Cu at (89.7, 32.4)
- added R63: 10R, Resistor_SMD:R_0402_1005Metric, F.Cu at (89.7, 34.6)
- added R64: 10R, Resistor_SMD:R_0402_1005Metric, F.Cu at (89.7, 36.7)
- added R65: 10R, Resistor_SMD:R_0402_1005Metric, F.Cu at (89.7, 38.8)
- added R66: 10R, Resistor_SMD:R_0402_1005Metric, F.Cu at (89.7, 33.5)
- added R67: 10R, Resistor_SMD:R_0402_1005Metric, F.Cu at (89.7, 35.6)
- added R68: 10R, Resistor_SMD:R_0402_1005Metric, F.Cu at (89.7, 37.7)
- added R7: 20k, Resistor_SMD:R_0402_1005Metric, F.Cu at (150.4, 44.1)
- added R8: 10k, Resistor_SMD:R_0402_1005Metric, F.Cu at (148.3, 44.1)
- added R9: 5.1k, Resistor_SMD:R_0402_1005Metric, F.Cu at (134.1, 89.1)
- added SW1: RESET, ASIC_Implementation_Library:PTS815SJM250SMTRLFS, F.Cu at (130.8, 30.8)
- added SW2: BOOT, ASIC_Implementation_Library:PTS815SJM250SMTRLFS, F.Cu at (101.2, 30.8)
- added TP1: TestPoint, TestPoint:TestPoint_Pad_1.0x1.0mm, F.Cu at (152.1, 66.1)
- added TP2: TestPoint, TestPoint:TestPoint_Pad_4.0x4.0mm, F.Cu at (163.3, 31.3)
- added TP3: TestPoint, TestPoint:TestPoint_Pad_4.0x4.0mm, F.Cu at (163.3, 51.5)
- added TP4: TestPoint, TestPoint:TestPoint_Pad_1.0x1.0mm, F.Cu at (82.4, 86.0)
- added U1: TMP117, Package_BGA:Texas_DSBGA-6_0.95x1.488mm_Layout2x3_P0.4mm, F.Cu at (104.9, 70.6)
- added U2: ~, ASIC_Implementation_Library:ESP32S2MINI1N4R2, F.Cu at (116.8, 38.8)
- added U3: USB4105, ASIC_Implementation_Library:USB4105, F.Cu at (140.6, 89.1)
Routing:
- net +3.3VA: track 0.00 -> 185.3 mm, vias 0 -> 9
- net Vref: track 0.00 -> 126.9 mm, vias 0 -> 6
- net -3V3: track 0.00 -> 92.6 mm, vias 0 -> 4
- net Stim_gnd: track 0.00 -> 85.4 mm, vias 0 -> 1
- net Stim+: track 0.00 -> 83.2 mm
- net Stim-: track 0.00 -> 81.7 mm
- net Istim: track 0.00 -> 59.5 mm
- net Stim_out: track 0.00 -> 55.4 mm, vias 0 -> 1
- net Probe_in_4+: track 0.00 -> 49.7 mm
- net ~{CS}: track 0.00 -> 45.4 mm, vias 0 -> 1
- net Probe_in_4-: track 0.00 -> 44.8 mm, vias 0 -> 1
- net Probe_in_1+: track 0.00 -> 43.0 mm, vias 0 -> 1
- net SCK: track 0.00 -> 42.5 mm, vias 0 -> 1
- net Probe_in_3+: track 0.00 -> 42.0 mm, vias 0 -> 1
- net Probe_in_2+: track 0.00 -> 41.5 mm, vias 0 -> 1
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Other:
- board outline added: 146.9 x 71.1 mm
- board text added: "+3.3V"
- board text added: "+3.3VA"
- board text added: "+9V"
- board text added: "-3.3VA"
- board text added: "-9V"
- board text added: "-VPOTECTION"
- board text added: "3.3V"
- board text added: "ADC"
- board text added: "ADC1"
- board text added: "ADC2"
- board text added: "ADC3"
- board text added: "ADC4"
- board text added: "AMP1"
- board text added: "AMP2"
- board text added: "AMP3"
- board text added: "AMP4"
- board text added: "ANALOG"
- board text added: "BATT"
- board text added: "BATTERY"
- board text added: "BOOT"
- board text added: "BYPASS"
- board text added: "CH1"
- board text added: "CH2"
- board text added: "COIL+"
- board text added: "COIL-"
- board text added: "DIGITAL"
- board text added: "FS"
- board text added: "GAUGE"
- board text added: "GND"
- board text added: "GPIO1"
- board text added: "GPIO10"
- board text added: "GPIO11"
- board text added: "GPIO12"
- board text added: "GPIO13"
- board text added: "GPIO14"
- board text added: "GPIO15"
- board text added: "GPIO16"
- board text added: "GPIO2"
- board text added: "GPIO3"
- board text added: "GPIO33"
- board text added: "GPIO34"
- board text added: "GPIO35"
- board text added: "GPIO36"
- board text added: "GPIO37"
- board text added: "GPIO38"
- board text added: "GPIO4"
- board text added: "GPIO45"
- board text added: "GPIO5"
- board text added: "GPIO6"
- board text added: "GPIO7"
- board text added: "GPIO8"
- board text added: "GPIO9"
- board text added: "HV"
- board text added: "IMEAS"
- board text added: "IN1+"
- board text added: "IN1-"
- board text added: "IN2+"
- board text added: "IN2-"
- board text added: "IN3+"
- board text added: "IN3-"
- board text added: "IN4+"
- board text added: "IN4-"
- board text added: "ISTIM GEN"
- board text added: "MCLK"
- board text added: "PGND"
- board text added: "PROBE"
- board text added: "RST"
- board text added: "RX"
- board text added: "SCK"
- board text added: "SCL"
- board text added: "SDA"
- board text added: "SDI"
- board text added: "SDO"
- board text added: "SEL"
- board text added: "SPI"
- board text added: "STIM"
- board text added: "SYS"
- board text added: "TEMP"
- board text added: "TX"
- board text added: "USB"
- board text added: "USB-C"
- board text added: "VAnalog"
- board text added: "VREF"
- board text added: "VSTIM"
- board text added: "VSYS"
- board text added: "WIRE"
- board text added: "WIRELESS POWER"
- board text added: "WS"
- board text added: "~{CS}"
- board text added: "~{IRQ}"
